File: Hardware/Rev 1.sch (EAGLE design)
At the start: 16 parts, among them IC1 LM5069MM-2, T1 AUIRFS8409-7P

Commit message: Add image and current limit maths.
Connections:
- net VIN: now also R3.2
- net VIN_K: no longer R3.2
Other:
- note added: "R1 = 55mV / Ilimit"
Changed lines of the file:
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@@
 <text x="71.12" y="77.47" size="1.778" layer="97">6S</text>
 <wire x1="38.1" y1="67.31" x2="38.1" y2="80.01" width="0.1524" layer="97"/>
+<text x="88.9" y="134.62" size="1.778" layer="97">R1 = 55mV / Ilimit</text>
 </plain>
 <instances>
@@
 <pinref part="R1" gate="G$1" pin="B1"/>
 <pinref part="R1" gate="G$1" pin="B2"/>
-<wire x1="91.44" y1="124.46" x2="58.42" y2="124.46" width="0.6096" layer="91"/>
+<wire x1="91.44" y1="124.46" x2="86.36" y2="124.46" width="0.6096" layer="91"/>
+<wire x1="86.36" y1="124.46" x2="58.42" y2="124.46" width="0.6096" layer="91"/>
 <wire x1="92.71" y1="127" x2="91.44" y2="127" width="0.6096" layer="91"/>
 <wire x1="91.44" y1="127" x2="91.44" y2="124.46" width="0.6096" layer="91"/>
@@
 <pinref part="PAD1" gate="1" pin="P"/>
 <label x="68.58" y="127" size="1.778" layer="95"/>
+<pinref part="R3" gate="G$1" pin="2"/>
+<wire x1="91.44" y1="99.06" x2="86.36" y2="99.06" width="0.1524" layer="91"/>
+<wire x1="86.36" y1="99.06" x2="86.36" y2="124.46" width="0.1524" layer="91"/>
+<junction x="86.36" y="124.46"/>
 </segment>
 <segment>
@@
 <wire x1="91.44" y1="121.92" x2="92.71" y2="121.92" width="0.1524" layer="91"/>
 <pinref part="C1" gate="G$1" pin="1"/>
-<pinref part="R3" gate="G$1" pin="2"/>
 <pinref part="IC1" gate="A" pin="VIN"/>
 <wire x1="109.22" y1="101.6" x2="91.44" y2="101.6" width="0.1524" layer="91"/>
-<wire x1="91.44" y1="101.6" x2="91.44" y2="99.06" width="0.1524" layer="91"/>
 <junction x="91.44" y="101.6"/>
 <wire x1="91.44" y1="101.6" x2="83.82" y2="101.6" width="0.1524" layer="91"/>
